File: kicad/ESP PogoPin Programmer.kicad_pcb (KiCad board)
At the start: 2 copper layers, 64.5 x 17.8 mm, 32 parts, among them J1 USB_B_Micro, J10 Conn_01x06, J2 ~Reset, J3 RxD, J4 TxD, J5 Enable, J6 Flash, J7 3V3, J8 GND, J9 ESP-01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

Commit message: minor
Parts:
- added J11: 3V3, barn53-kicad:PogoPin_vertical, F.Cu at (131.1, 117.9)
- added J12: GND, barn53-kicad:PogoPin_vertical, F.Cu at (133.3, 117.9)
- added R8: 10k, Resistor_SMD:R_0805_2012Metric, F.Cu at (132.1, 115.2)
- added R9: 10k, Resistor_SMD:R_0805_2012Metric, F.Cu at (136.5, 115.2)
- J3: value RxD -> TxD
- J4: value TxD -> RxD
- J7: value 3V3 -> GPIO2
- J8: value GND -> GPIO15
Connections:
- J7 pad 1: /3V3 -> /GPIO2
- J8 pad 1: GND -> /GPIO15
- J9 pad 3: Net-(J9-Pad3) -> /GPIO2
